Commit message: feat: fix config for benchmark
Created seperate config files for benchmark so that the config files can be chaged for different robot

File: urdf/udacity_bot_long.xacro (robot description, xacro)
@@ -8,5 +8,5 @@
     <child link="chassis" />
   </joint>
-  <!-- Robot chasis and caste wheels -->
+  <!-- Robot chasis -->
   <link name='chassis'>
     <pose>0 0 0.1 0 0 0</pose>
@@ -19,17 +19,26 @@
     </inertial>
     <collision name='collision'>
-      <origin xyz="0 0 0" rpy=" 0 0 0"/>
+      <origin xyz="-0.2 0 0" rpy=" 0 0 0"/>
       <geometry>
-        <box size=".4 .6 .1"/>
+        <box size=".8 .2 .1"/>
       </geometry>
     </collision>
     <visual name='chassis_visual'>
-      <origin xyz="0 0 0" rpy=" 0 0 0"/>
+      <origin xyz="-0.2 0 0" rpy=" 0 0 0"/>
       <geometry>
-        <box size=".4 .6 .1"/>
+        <box size=".8 .2 .1"/>
       </geometry>
     </visual>
+  </link>
+  <link name='caste_wheel'>
+   <inertial>
+      <mass value="2.0"/>
+      <origin xyz="0.0 0 0" rpy=" 0 0 0"/>
+      <inertia ixx="0.1" ixy="0" ixz="0"
+                iyy="0.1" iyz="0"
+                izz="0.1" />
+    </inertial>
     <collision name='back_caster_collision'>
-      <origin xyz="-0.15 0 -0.05" rpy=" 0 0 0"/>
+      <origin xyz="0 0 0" rpy=" 0 0 0"/>
       <geometry>
         <sphere radius="0.0499"/>
@@ -37,22 +46,29 @@
     </collision>
     <visual name='back_caster_visual'>
-      <origin xyz="-0.15 0 -0.05" rpy=" 0 0 0"/>
+      <origin xyz="0 0 0" rpy=" 0 0 0"/>
       <geometry>
         <sphere radius="0.05"/>
       </geometry>
     </visual>
-    <collision name='front_caster_collision'>
-      <origin xyz="0.15 0 -0.05" rpy=" 0 0 0"/>
+<!--
+    <collision name='back_right_caster_collision'>
+      <origin xyz="-0.55 0.06 -0.05" rpy=" 0 0 0"/>
       <geometry>
         <sphere radius="0.0499"/>
       </geometry>
     </collision>
-    <visual name='front_caster_visual'>
-      <origin xyz="0.15 0 -0.05" rpy=" 0 0 0"/>
+    <visual name='back_right_caster_visual'>
+      <origin xyz="-0.55 0.06 -0.05" rpy=" 0 0 0"/>
       <geometry>
         <sphere radius="0.05"/>
       </geometry>
     </visual>
+-->
   </link>
+    <joint name="caste_joint" type="fixed">
+      <origin xyz="-0.55 0 -0.05" rpy="0 0 0" />
+      <parent link="chassis"/>
+      <child link="caste_wheel" />
+    </joint>
     <!-- Macro for creating wheel links -->
    <xacro:macro name="wheel" params="name">
@@ -85,5 +101,5 @@
    <!-- Creating wheel joints -->
    <joint type="continuous" name="left_wheel_hinge">
-     <origin xyz="0 0.35 0" rpy="0 0 0"/>
+     <origin xyz="0 0.15 0" rpy="0 0 0"/>
      <child link="left_wheel"/>
      <parent link="chassis"/>
@@ -93,5 +109,5 @@
    </joint>
    <joint type="continuous" name="right_wheel_hinge">
-      <origin xyz="0 -0.35 0" rpy="0 0 0"/>
+      <origin xyz="0 -0.15 0" rpy="0 0 0"/>
       <child link="right_wheel"/>
       <parent link="chassis"/>
