Commit message: feat: fix laser range finder wheel detection bug
Changed the minimum range of the laser range finder to be 0.15 so that the wheels are not detected as obsticles

File: urdf/benchmark/udacity_bot_benchmark.xacro (robot description, xacro)
@@ -152,5 +152,5 @@
     </link>
     <joint name="hokuyo_joint" type="fixed">
-      <origin xyz="0.2 0 0.1" rpy="0 0 0" />
+      <origin xyz="0.15 0 0.1" rpy="0 0 0" />
       <parent link="chassis"/>
       <child link="hokuyo" />

Commit message: feat: Change min laser distance for wide robot Changed the min value for the laser range finder in the udacity_bot.gazebo file and also made sure that the benchmark was not effected

File: urdf/benchmark/udacity_bot_benchmark.xacro (robot description, xacro)
@@ -1,5 +1,5 @@
 <?xml version='1.0'?>
 <robot name="udacity_bot" xmlns:xacro="http://www.ros.org/wiki/xacro">
-  <xacro:include filename="$(find udacity_bot)/urdf/udacity_bot.gazebo" />
+  <xacro:include filename="$(find udacity_bot)/urdf/benchmark/udacity_bot_benchmark.gazebo" />
 <link name="robot_footprint"></link>
   <joint name="robot_footprint_joint" type="fixed">

File: urdf/udacity_bot.xacro (robot description, xacro)
@@ -152,5 +152,5 @@
     </link>
     <joint name="hokuyo_joint" type="fixed">
-      <origin xyz="0.15 0 0.1" rpy="0 0 0" />
+      <origin xyz="0.0 0 0.2" rpy="0 0 0" />
       <parent link="chassis"/>
       <child link="hokuyo" />
